Commit message: change grippers to LND and optimize the corresponding collision geometry used in URDF file; modify waypoints to enable rl demos

File: surrol/assets/psm/psm.urdf (robot description, URDF)
Before this commit: robot psm, 17 links, 16 joints
Links:
- link psm_tool_gripper1_link: geometry collision mesh filename=meshes/collision/LND_Jaw_rotated_L_vhacd.obj scale=0.001 0.001 0.001; visual mesh filename=meshes/visual/LND_Jaw_rotated_L.obj scale=0.001 0.001 0.001
- link psm_tool_gripper2_link: geometry collision mesh filename=meshes/collision/LND_Jaw_rotated_R_vhacd.obj scale=0.001 0.001 0.001; visual mesh filename=meshes/visual/LND_Jaw_rotated_R.obj scale=0.001 0.001 0.001
