Commit message: solve interpenetration problem btw objects and related issues(rl_demo failure, ecm out of control, yaw_control) add border collision for tray pad; change grippers and shaft, add contact constraint for stable grasping; add new tasks: needle the rings and pegboard; change floor

File: surrol/assets/block/block.urdf (robot description, URDF)
Before this commit: robot block, 4 links, 3 joints
Links:
- link baseLink: mass 0.01 -> 1.01

File: surrol/assets/needle/needle_40mm.urdf (robot description, URDF)
Before this commit: robot needle, 7 links, 6 joints
Links:
- link baseLink: mass 0.01 -> 0.51

File: surrol/assets/peg_board/peg_board.urdf (robot description, URDF)
Before this commit: robot peg_board, 13 links, 12 joints
Links:
- link baseLink: mass .0 -> 100.0
- link peg_1: mass .0 -> 100.0
- link peg_10: mass .0 -> 100.0
- link peg_11: mass .0 -> 100.0
- link peg_12: mass .0 -> 100.0
- link peg_2: mass .0 -> 100.0
- link peg_3: mass .0 -> 100.0
- link peg_4: mass .0 -> 100.0
- link peg_5: mass .0 -> 100.0
- link peg_6: mass .0 -> 100.0
- link peg_7: mass .0 -> 100.0
- link peg_8: mass .0 -> 100.0
- link peg_9: mass .0 -> 100.0

File: surrol/assets/psm/psm.urdf (robot description, URDF)
Before this commit: robot psm, 17 links, 16 joints
Links:
- link psm_main_insertion_link_3: geometry visual mesh filename=meshes/visual/CDF_base.obj scale=0.001 0.001 0.001
- link psm_tool_gripper1_link: mass 0.02 -> 2.02; geometry collision mesh filename=meshes/collision/yaw1_vhacd.obj scale=0.0005 0.0005 0.0005; visual mesh filename=meshes/visual/yaw1.obj scale=0.0005 0.0005 0.0005
- link psm_tool_gripper2_link: mass 0.02 -> 2.02; geometry collision mesh filename=meshes/collision/yaw2_vhacd.obj scale=0.0005 0.0005 0.0005; visual mesh filename=meshes/visual/yaw2.obj scale=0.0005 0.0005 0.0005
- link psm_tool_pitch_link: geometry collision mesh filename=meshes/collision/wrist.obj scale=0.001 0.001 0.001; visual mesh filename=meshes/visual/wrist.obj scale=0.001 0.001 0.001
- link psm_tool_roll_link: geometry collision mesh filename=meshes/collision/CDF_base_no_shaft.obj scale=0.001 0.001 0.001; visual mesh filename=meshes/visual/CDF_base_no_shaft.obj scale=0.001 0.001 0.001
- link psm_tool_yaw_link: geometry 
Joints:
- joint psm_main_insertion_joint: limit lower=0 upper=0.24 effort=100 velocity=1 -> lower=0 upper=0.24 effort=200 velocity=1
- joint psm_pitch_back_joint: limit lower=-0.93556 upper=0.94249 effort=100 velocity=10 -> lower=-0.93556 upper=0.94249 effort=200 velocity=10
- joint psm_pitch_bottom_joint: limit lower=-0.94249 upper=0.93556 effort=100 velocity=10 -> lower=-0.94249 upper=0.93556 effort=200 velocity=10
- joint psm_pitch_end_joint: limit lower=-0.9251 upper=0.9251 effort=100 velocity=2.1 -> lower=-0.9251 upper=0.9251 effort=200 velocity=2.1
- joint psm_pitch_front_joint: limit lower=-0.93556 upper=0.94249 effort=100 velocity=10 -> lower=-0.93556 upper=0.94249 effort=200 velocity=10
- joint psm_pitch_top_joint: limit lower=-0.94249 upper=0.93556 effort=100 velocity=10 -> lower=-0.94249 upper=0.93556 effort=200 velocity=10
- joint psm_tool_gripper1_joint: limit lower=-1 upper=1 effort=20 velocity=2.1 -> lower=-1 upper=1 effort=200 velocity=2.1
- joint psm_tool_gripper2_joint: limit lower=-1 upper=1 effort=20 velocity=2.1 -> lower=-1 upper=1 effort=200 velocity=2.1
- joint psm_tool_pitch_joint: limit lower=-1.3963 upper=1.3963 effort=100 velocity=2.1 -> lower=-1.3963 upper=1.3963 effort=200 velocity=2.1
- joint psm_tool_roll_joint: limit lower=-4.5379 upper=4.5379 effort=100 velocity=2.1 -> lower=-4.5379 upper=4.5379 effort=200 velocity=2.1
- joint psm_tool_yaw_joint: limit lower=-1.3963 upper=1.3963 effort=100 velocity=2.1 -> lower=-1.3963 upper=1.3963 effort=200 velocity=21
- joint psm_yaw_joint: limit lower=-1.5883 upper=1.5883 effort=100 velocity=2.1 -> lower=-1.5883 upper=1.5883 effort=200 velocity=2.1

File: surrol/assets/ring/ring.urdf (robot description, URDF)
Before this commit: robot ring, 7 links, 6 joints
Links:
- link baseLink: mass 0.01 -> 100.01

File: surrol/assets/tray/tray_pad.urdf (robot description, URDF)
Before this commit: robot tray, 6 links, 5 joints
Links:
- link baseLink: mass .0 -> 100.0
- link border_1: mass .0 -> 100.0; geometry collision box size=0.120 0.003 0.025; visual box size=0 0 0
- link border_2: mass .0 -> 100.0; geometry collision box size=0.120 0.003 0.025; visual box size=0 0 0
- link border_3: mass .0 -> 100.0; geometry collision box size=0.003 0.196 0.025; visual box size=0 0 0
- link border_4: mass .0 -> 100.0; geometry collision box size=0.003 0.196 0.025; visual box size=0 0 0
- link pad: mass .0 -> 100.0

Commit message: change grippers to LND and optimize the corresponding collision geometry used in URDF file; modify waypoints to enable rl demos

File: surrol/assets/block/block.urdf (robot description, URDF)
Before this commit: robot block, 4 links, 3 joints
Links:
- link baseLink: mass 1.01 -> 2.01

File: surrol/assets/psm/psm.urdf (robot description, URDF)
Before this commit: robot psm, 17 links, 16 joints
Links:
- link psm_tool_gripper1_link: geometry collision mesh filename=meshes/collision/LND_Jaw_L_vhacd_512_500k.obj scale=0.001 0.001 0.001; visual mesh filename=meshes/visual/LND_Jaw_L.obj scale=0.001 0.001 0.001
- link psm_tool_gripper2_link: geometry collision mesh filename=meshes/collision/LND_Jaw_R_vhacd_512_500k.obj scale=0.001 0.001 0.001; visual mesh filename=meshes/visual/LND_Jaw_R.obj scale=0.001 0.001 0.001

Commit message: 1.add new tasks: pick and place; match board; 2. modify previous tasks to enable haptic demo data collection for rl training 3. integrate two rl learnt policies into the simulator(demo_rl_scenes.py) 4. solve unexpected peg moving problem which occured after introducing constraints for stable grasping(caused by redundant waypoint link)

File: surrol/assets/block/block.urdf (robot description, URDF)
Before this commit: robot block, 4 links, 3 joints
Links:
- link baseLink: mass 2.01 -> 2.5

File: surrol/assets/psm/psm.urdf (robot description, URDF)
Before this commit: robot psm, 17 links, 16 joints
Links:
- link psm_tool_gripper1_link: geometry collision box size=0.0014 0.0102 0.0018; visual mesh filename=meshes/visual/tool_gripper1_link_wide.obj
- link psm_tool_gripper2_link: geometry collision box size=0.0014 0.0102 0.0018; visual mesh filename=meshes/visual/tool_gripper2_link_wide.obj
