Commit message: Record demonstration

File: surrol/assets/block/block_haptic.urdf (robot description, URDF)
Before this commit: robot block, 1 links, 0 joints
Links:
- link baseLink: mass 2.5 -> 0.5

File: surrol/assets/peg_board/peg_board.urdf (robot description, URDF)
Before this commit: robot peg_board, 13 links, 12 joints
Links:
- link peg_1: geometry collision cylinder length=0.0168 radius=0.001; visual mesh filename=meshes/peg.obj scale=1 1 0.6
- link peg_10: geometry collision cylinder length=0.0168 radius=0.001; visual mesh filename=meshes/peg.obj scale=1 1 0.6
- link peg_11: geometry collision cylinder length=0.0168 radius=0.001; visual mesh filename=meshes/peg.obj scale=1 1 0.6
- link peg_12: geometry collision cylinder length=0.0168 radius=0.001; visual mesh filename=meshes/peg.obj scale=1 1 0.6
- link peg_2: geometry collision cylinder length=0.0168 radius=0.001; visual mesh filename=meshes/peg.obj scale=1 1 0.6
- link peg_3: geometry collision cylinder length=0.0168 radius=0.001; visual mesh filename=meshes/peg.obj scale=1 1 0.6
- link peg_4: geometry collision cylinder length=0.0168 radius=0.001; visual mesh filename=meshes/peg.obj scale=1 1 0.6
- link peg_5: geometry collision cylinder length=0.0168 radius=0.001; visual mesh filename=meshes/peg.obj scale=1 1 0.6
- link peg_6: geometry collision cylinder length=0.0168 radius=0.001; visual mesh filename=meshes/peg.obj scale=1 1 0.6
- link peg_7: geometry collision cylinder length=0.0168 radius=0.001; visual mesh filename=meshes/peg.obj scale=1 1 0.6
- link peg_8: geometry collision cylinder length=0.0168 radius=0.001; visual mesh filename=meshes/peg.obj scale=1 1 0.6
- link peg_9: geometry collision cylinder length=0.0168 radius=0.001; visual mesh filename=meshes/peg.obj scale=1 1 0.6

File: surrol/assets/pegboard/lower_nut.urdf (robot description, URDF)
Before this commit: robot board, 1 links, 0 joints
Links:
- link baseLink: geometry collision mesh filename=meshes/lower_nut.obj scale=0.75 0.75 0.75; visual mesh filename=meshes/lower_nut.obj scale=0.75 0.75 0.75

File: surrol/assets/pegboard/lower_peg.urdf (robot description, URDF)
Before this commit: robot board, 1 links, 0 joints
Links:
- link baseLink: geometry collision mesh filename=meshes/lower_peg_collision.obj scale=0.75 0.75 0.75; visual mesh filename=meshes/lower_peg.obj scale=0.75 0.75 0.75

File: surrol/assets/pegboard/upper_nut.urdf (robot description, URDF)
Before this commit: robot board, 1 links, 0 joints
Links:
- link baseLink: geometry collision mesh filename=meshes/upper_nut.obj scale=0.75 0.75 0.75; visual mesh filename=meshes/upper_nut.obj scale=0.75 0.75 0.75

File: surrol/assets/pegboard/upper_peg.urdf (robot description, URDF)
Before this commit: robot board, 1 links, 0 joints
Links:
- link baseLink: geometry collision mesh filename=meshes/upper_peg_collision.obj scale=0.75 0.75 0.75; visual mesh filename=meshes/upper_peg.obj scale=0.75 0.75 0.75

File: surrol/assets/tray/tray_pad.urdf (robot description, URDF)
Before this commit: robot tray, 6 links, 5 joints
Links:
- link baseLink: mass 100.0 -> 0.01
- link pad: mass 100.0 -> 0.01
