Commit message: enable ECM stereo display

File: surrol/assets/CH4/CH4_waypoints.urdf (robot description, URDF)
Before this commit: robot ring, 7 links, 6 joints
Links:
- removed link waypoint_2
- removed link waypoint_3
- removed link waypoint_4
- removed link waypoint_5
Joints:
- removed joint waypoint_joint_2
- removed joint waypoint_joint_3
- removed joint waypoint_joint_4
- removed joint waypoint_joint_5
- joint waypoint_joint_1: origin xyz=-0.02 0 0 rpy=0 0 0 -> xyz=0 0.01 0 rpy=0 0 0

File: surrol/assets/block/block.urdf (robot description, URDF)
Before this commit: robot block, 4 links, 3 joints
Links:
- link baseLink: mass 2.5 -> 1

File: surrol/assets/ring_cyl/ring_cyl.urdf (robot description, URDF)
Before this commit: robot needle, 7 links, 6 joints
Links:
- link baseLink: mass 0.51 -> 0.01; geometry collision mesh filename=meshes/ring_cyl_vhacd.obj scale=1 1 1; visual mesh filename=meshes/ring_cyl.obj scale=1 1 1

File: surrol/assets/ring_cyl/ring_cyl_red.urdf (robot description, URDF)
Before this commit: robot needle, 7 links, 6 joints
Links:
- link baseLink: mass 0.51 -> 0.01; geometry collision mesh filename=meshes/ring_cyl_vhacd.obj scale=1 1 1; visual mesh filename=meshes/ring_cyl.obj scale=1 1 1

File: surrol/assets/ring_cyl/ring_cyl_yellow.urdf (robot description, URDF)
Before this commit: robot needle, 7 links, 6 joints
Links:
- link baseLink: mass 0.51 -> 0.01; geometry collision mesh filename=meshes/ring_cyl_vhacd.obj scale=1 1 1; visual mesh filename=meshes/ring_cyl.obj scale=1 1 1
