Commit message: stable

File: surrol/assets/CH4/CH4.urdf (robot description, URDF)
Before this commit: robot ring, 1 links, 0 joints
Links:
- link baseLink: mass 2.01 -> 0.5

File: surrol/assets/CH4/CH4_waypoints.urdf (robot description, URDF)
Before this commit: robot ring, 3 links, 2 joints
Links:
- link baseLink: mass 2.01 -> 0.5

File: surrol/assets/match_board/0.urdf (robot description, URDF)
Before this commit: robot ring, 1 links, 0 joints
Links:
- link baseLink: mass 1.01 -> 0.5

File: surrol/assets/match_board/1.urdf (robot description, URDF)
Before this commit: robot ring, 1 links, 0 joints
Links:
- link baseLink: mass 2.01 -> 0.5

File: surrol/assets/match_board/2.urdf (robot description, URDF)
Before this commit: robot ring, 1 links, 0 joints
Links:
- link baseLink: mass 2.01 -> 0.5

File: surrol/assets/match_board/4.urdf (robot description, URDF)
Before this commit: robot ring, 1 links, 0 joints
Links:
- link baseLink: mass 2.01 -> 0.5

File: surrol/assets/match_board/5.urdf (robot description, URDF)
Before this commit: robot ring, 1 links, 0 joints
Links:
- link baseLink: mass 2.01 -> 0.5

File: surrol/assets/match_board/6.urdf (robot description, URDF)
Before this commit: robot ring, 1 links, 0 joints
Links:
- link baseLink: mass 2.01 -> 0.5

File: surrol/assets/match_board/a.urdf (robot description, URDF)
Before this commit: robot ring, 1 links, 0 joints
Links:
- link baseLink: mass 2.01 -> 0.5

File: surrol/assets/match_board/b.urdf (robot description, URDF)
Before this commit: robot ring, 1 links, 0 joints
Links:
- link baseLink: mass 2.01 -> 0.5

File: surrol/assets/match_board/c.urdf (robot description, URDF)
Before this commit: robot ring, 1 links, 0 joints
Links:
- link baseLink: mass 2.01 -> 0.5
